Commit message: added rviz feature, cleaned up controller code

File: robot_resources/desktop_arm_description/urdf/desktop_arm.urdf (robot description, URDF)
Before this commit: robot desktop_arm_description, 7 links, 6 joints
Links:
- added link base
- added link tool0
Joints:
- removed joint joint_0
- added joint base_link-base: type fixed, parent base_link, child base, origin xyz=0 0 0 rpy=0 0 0
- added joint joint6-tool0: type fixed, parent end_effector, child tool0, origin xyz=0 0 0 rpy=0 0.5 0
- added joint joint_6: type revolute, parent link_5, child end_effector, origin xyz=0.17605 0.29813 -0.29218 rpy=1.1615 0.33095 -2.9233, axis 0 0 0
- joint joint_1: axis 0.934125217802764 0 0.356945482482884 -> 0 1 0; child link_2 -> link_1; origin xyz=0 0.1655 0 rpy=0.288567690879059 -0.0158462661982318 0.10895820907763 -> xyz=0.0320497775774861 -0.156148136610897 0.0881843828733705 rpy=1.5707963267949 0 0.70838946909971; parent link_1 -> base_link
- joint joint_2: axis 0.934125217802763 0 0.356945482482886 -> 0.934125217802764 0 0.356945482482884; child link_3 -> link_2; origin xyz=0.0533123755144546 0.163058763880744 -0.139518320956508 rpy=-0.28856769087906 -0.0158462661982266 -0.10895820907763 -> xyz=0 0.1655 0 rpy=0.288567690879059 -0.0158462661982318 0.10895820907763; parent link_2 -> link_1
- joint joint_3: axis 0.33384 0.35396 -0.87365 -> 0.934125217802763 0 0.356945482482886; child link_4 -> link_3; origin xyz=0.039132 0.040964 -0.10092 rpy=-0.81888 0.68462 3.0043 -> xyz=0.0533123755144546 0.163058763880744 -0.139518320956508 rpy=-0.28856769087906 -0.0158462661982266 -0.10895820907763; parent link_3 -> link_2
- joint joint_4: axis 0.9426 -0.13293 0.30633 -> 0.33384 0.35396 -0.87365; child link_5 -> link_4; origin xyz=0.035644 0.037793 -0.09328 rpy=0.99317 -0.27115 0.21303 -> xyz=0.039132 0.040964 -0.10092 rpy=-0.81888 0.68462 3.0043; parent link_4 -> link_3
- joint joint_5: axis 0 0 0 -> 0.9426 -0.13293 0.30633; child end_effector -> link_5; limit (none) -> lower=-1.3 upper=1.3 effort=0 velocity=0; origin xyz=0.17605 0.29813 -0.29218 rpy=1.1615 0.33095 -2.9233 -> xyz=0.035644 0.037793 -0.09328 rpy=0.99317 -0.27115 0.21303; parent link_5 -> link_4; type fixed -> revolute

Commit message: joint state publishing, right now just the first joint

File: robot_resources/desktop_arm_description/urdf/desktop_arm.urdf (robot description, URDF)
Before this commit: robot desktop-arm, 9 links, 8 joints
Links:
- removed link base
- removed link tool0
Joints:
- removed joint base_link-base
- removed joint joint6-tool0
- joint joint_6: type revolute -> fixed
